File: LongHornNeonSign.kicad_pcb (KiCad board)
At the start: 2 copper layers, 83.5 x 70.2 mm, 65 parts, among them J1 Screw_Terminal_01x02, J2 Screw_Terminal_01x02, J3 Screw_Terminal_01x02, J4 Screw_Terminal_01x02, M1 MountingHole_3.2mm_M3, Q1 AO3400A, Q2 AO3400A, Q3 AO3400A, Q4 AO3400A, SW1 SW_Push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

Commit message: May 12 2026 run it back
Parts:
- COUT1: footprint Capacitor_SMD:CP_Elec_8x10 -> Capacitor_SMD:CP_Elec_6.3x7.7
- moved COUT1 1.42 mm to (176.3, 97.4)
- moved BJ_C1 0.88 mm to (185.4, 122.8)
Routing:
- net /+5V: track 99.8 -> 100.4 mm
- net GND: vias 129 -> 128
Other:
- board text added: "LONGHORN Neon Sign Jennifer Li 12V Max v1.0"
