File: LongHornNeonSign.kicad_sch (KiCad schematic)
At the start: 61 parts, among them J1 Barrel_Jack, J2 Screw_Terminal_01x02, J3 Screw_Terminal_01x02, J4 Screw_Terminal_01x02, J5 Screw_Terminal_01x02, Q1 AO3400A, Q2 AO3400A, Q3 AO3400A, Q4 AO3400A, SW1 SW_Push, SW2 SW_Push, SW3 SW_Push, U1 LM2596S-5

Commit message: update
Parts:
- L_12V1: renamed from LED_12V1; value DL_12V -> 12V
- L_5V1: renamed from LED_5V1; value DL_5V -> 5V
- L_A0: renamed from LED_5V4; value DL_D9 -> A0
- L_A1: renamed from LED_5V5; value DL_D10 -> A1
- L_A2: renamed from LED_5V6; value DL_D11 -> A2
- L_A3: renamed from LED_5V7; value DL_D12 -> A3
- L_D0: renamed from LED_5V2; value DL_D0 -> D0
- L_D1: renamed from LED_5V3; value DL_D1 -> D1
- L_D13: renamed from LED_5V8; value DL_D13 -> D13
- TP_DOWN1: value BTN_DOWN -> DOWN
- TP_PWM1: value PWM_OUT1 -> PWM1
- TP_PWM2: value PWM_OUT2 -> PWM2
- TP_PWM3: value PWM_OUT3 -> PWM3
- TP_PWM4: value PWM_OUT4 -> PWM4
- TP_TOG1: value BTN_TOGGLE -> TOGGLE
- TP_UP1: value BTN_UP -> UP
- renumbered J1 to BJ_C1, C_DEBOUNCE1 to DBC1, C_DEBOUNCE2 to DBC2, C_DEBOUNCE3 to DBC3, C_DECOUP1 to DCC1, D2 to Diode1, J2 to J1, J3 to J2, J4 to J3, J5 to J4, R1 to R_12V1, R2 to R_5V1, R5 to R_A0, R6 to R_A1, R7 to R_A2, R8 to R_A3, R3 to R_D0, R4 to R_D1, R9 to R_D13, R_PD7 to R_PD4, R_PD4 to R_PD5, R_PD5 to R_PD6, R_PD6 to R_PD7, TP12V1 to TP_12V1, TP5V1 to TP_5V1, TPGND1 to TP_GND1
Connections:
- net BTN_DOWN renamed DOWN
- net BTN_TOGGLE renamed TOG
- net BTN_UP renamed UP
- net D_DEBUG0 renamed D_D0
- net D_DEBUG1 renamed D_D1
- net D_DEBUG10 renamed D_A1
- net D_DEBUG11 renamed D_A2
- net D_DEBUG12 renamed D_A3
- net D_DEBUG13 renamed D_D13
- net D_DEBUG9 renamed D_A0
- net PWM_OUT1 renamed PWM1
- net PWM_OUT2 renamed PWM2
- net PWM_OUT3 renamed PWM3
- net PWM_OUT4 renamed PWM4

Commit message: May 12 2026 run it back
Parts:
- COUT1: footprint Capacitor_SMD:CP_Elec_8x10 -> Capacitor_SMD:CP_Elec_6.3x7.7; LCSC C976031 -> C2827940
Changed lines of the file:
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@@
 			)
 		)
-		(property "Footprint" "Capacitor_SMD:CP_Elec_8x10"
+		(property "Footprint" "Capacitor_SMD:CP_Elec_6.3x7.7"
 			(at 130.5052 118.11 0)
 			(effects
@@
 			)
 		)
-		(property "LCSC" "C976031"
+		(property "LCSC" "C2827940"
 			(at 129.54 114.3 0)
 			(effects
@@
 		(on_board yes)
 		(dnp no)
-		(fields_autoplaced yes)
 		(property "Reference" "#PWR031"
 			(at 85.09 101.6 0)
@@
 		)
 		(property "Value" "+12V"
-			(at 77.47 101.5999 90)
-			(effects
-				(font
+			(at 77.724 101.6 90)
+			(effects
+				(font
