File: Hardware/LongHornNeonSign.kicad_pcb (KiCad board)
At the start: 2 copper layers, 37 x 59.2 mm, 58 parts, among them J1 Barrel_Jack_Switch, J2 Screw_Terminal_01x02, J5 Screw_Terminal_01x02, Q1 AO3400A, Q4 AO3400A, U1 LMR34215FSC5RNXRQ1

Commit message: finalize PCB, added images and silkscreen text and 3D models
Parts:
- added G***: LOGO, LOGO, F.Cu at (149.1, 90.5)
- added G***: LOGO, LOGO, F.Cu at (149.0, 75.1)
- added G***: LOGO, LOGO, F.Cu at (120.8, 114.8)
- added G***: LOGO, LOGO, F.Cu at (149.3, 110.4)
- added G***: LOGO, LOGO, F.Cu at (145.9, 110.4)
- added G***: LOGO, LOGO, F.Cu at (123.3, 72.2)
- added G***: LOGO, LOGO, F.Cu at (122.5, 77.1)
- added G***: LOGO, LOGO, F.Cu at (145.1, 72.4)
- added G***: LOGO, LOGO, F.Cu at (120.2, 75.7)
- added G***: LOGO, LOGO, F.Cu at (147.3, 90.2)
- added G***: LOGO, LOGO, F.Cu at (122.2, 110.3)
- added G***: LOGO, LOGO, F.Cu at (124.3, 114.0)
- added G***: LOGO, LOGO, F.Cu at (153.8, 116.8)
- added G***: LOGO, LOGO, F.Cu at (149.2, 112.9)
- moved R2 2.95 mm to (122.8, 106.3), turned to 0 degrees
- moved D2 1.69 mm to (122.8, 107.4), turned to 0 degrees
- moved D1 1.47 mm to (136.4, 126.7)
- moved TP3 1.01 mm to (139.2, 126.9)
- moved R1 0.84 mm to (137.5, 127.1)
- moved D5 0.72 mm to (121.6, 89.6)
- moved TP4 0.44 mm to (122.8, 104.7)
Routing:
- net Net-(D1-A): track 1.75 -> 3.30 mm
- net +5V: track 68.8 -> 67.5 mm
- net Net-(D2-A): track 1.96 -> 3.15 mm
- net GND: track 2.80 -> 3.12 mm, vias 132 -> 136
Other:
- board text added: "+12V"
- board text added: "+5V"
- board text added: "HB"
