File: Hardware/LongHornNeonSign.kicad_sch (KiCad schematic)
At the start: 19 parts, among them J1 Barrel_Jack_Switch

Commit message: push RevB's README and edit schematic specs
Other:
- title: (none) -> Neon Sign PCB
Changed lines of the file:
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@@
 	(generator_version "9.0")
 	(paper "A4")
+	(title_block
+		(title "Neon Sign PCB")
+		(rev "RevB")
+	)
 	(rectangle
 		(start 144.78 182.88)
